File: kicad/kicad.kicad_sch (KiCad schematic)
At the start: 5 parts, among them U1 ESP32-c3 super mini, U2 VL53LDK, U3 VL53LDK

Commit message: added battery to kicad schematic
Parts:
- added BT1: 3V, symbol Device:Battery_Cell
Connections:
- net at U2. (X): now also U1.3
- net at U3. (X): now also U1.2
- new net: BT1.1 (+), U1. (GND), U2. (X), U3. (X)
- new net: BT1.2 (-), BZ1.2 (-), U1. (GND), U2. (X), U3. (X)
- new net: U1.8 (SDA), U2. (X), U3. (X)
- new net: U1.9 (SCL), U2. (X), U3. (X)
- now unconnected: U1. (GND), U1. (GND)
Changed lines of the file:
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@@
 		(title "Schemat połączeń w okularach")
 		(date "2025-03-11")
-		(comment 1 "Zasilanie poprzez port USB-C na ESP32-c3 (nie zawarty w schemacie)")
+		(comment 1 "programowanie poprzez port USB-C na ESP32-c3 (nie zawarty w schemacie)")
 	)
 	(junction
@@
 	)
 	(junction
+		(at 127 67.31)
+		(diameter 0)
+		(color 0 0 0 0)
+	)
+	(junction
+		(at 123.19 71.12)
+		(diameter 0)
+		(color 0 0 0 0)
+	)
+	(junction
 		(at 160.02 124.46)
 		(diameter 0)
@@
 	(wire
 		(pts
+			(xy 123.19 71.12) (xy 135.89 71.12)
+		)
+		(stroke
+			(width 0)
+			(type default)
+		)
+	)
+	(wire
+		(pts
 			(xy 64.77 128.27) (xy 163.83 128.27)
 		)
@@
 		(pts
 			(xy 186.69 138.43) (xy 186.69 116.84)
+		)
+		(stroke
+			(width 0)
+			(type default)
+		)
+	)
+	(wire
+		(pts
+			(xy 135.89 71.12) (xy 135.89 67.31)
+		)
+		(stroke
+			(width 0)
+			(type default)
+		)
+	)
+	(wire
+		(pts
+			(xy 135.89 67.31) (xy 134.62 67.31)
 		)
 		(stroke
@@
 	)
 	(symbol
-		(lib_name "okulary_parts:VL53LDK")
 		(lib_id "okulary_parts:VL53LDK")
 		(at 152.4 88.9 0)
@@
 	)
 	(symbol
-		(lib_name "okulary_parts:VL53LDK")
 		(lib_id "okulary_parts:VL53LDK")
 		(at 182.88 88.9 0)
@@
 					(unit 1)
 				)
+			)
+		)
+	)
+	(symbol
+		(lib_id "Device:Battery_Cell")
+		(at 129.54 67.31 270)
+		(unit 1)
+		(exclude_from_sim no)
+		(in_bom yes)
+		(on_board yes)
+		(dnp no)
+		(property "Reference" "BT1"
+			(at 131.3815 59.69 90)
+			(effects
+				(font
+					(size 1.27 1.27)
+				)
+			)
+		)
+		(property "Value" "3V"
+			(at 131.3815 62.23 90)
+			(effects
+				(font
+					(size 1.27 1.27)
+				)
+			)
+		)
+		(property "Footprint" ""
+			(at 131.064 67.31 90)
+			(effects
+				(font
+					(size 1.27 1.27)
+				)
+				(hide yes)
+			)
+		)
+		(property "Datasheet" "~"
+			(at 131.064 67.31 90)
+			(effects
+				(font
+					(size 1.27 1.27)
+				)
+				(hide yes)
+			)
+		)
+		(property "Description" "Single-cell battery"
+			(at 129.54 67.31 0)
+			(effects
+				(font
+					(size 1.27 1.27)
+				)
+				(hide yes)
+			)
+		)
+		(pin "2"
+		)
+		(pin "1"
+		)
+		(instances
+			(project ""
+				(path "/e697d9f0-6df0-4ad6-b7b8-3236f8a796fa"
+					(reference "BT1")
+					(unit 1)
+				)

Commit message: updated schematic
Parts:
- added U4: LM78L05_TO92, Package_TO_SOT_THT:TO-92_Inline, symbol Regulator_Linear:LM78L05_TO92
- BT1: value 3V -> 12V
Connections:
- net at U2. (X): now also U1.3
- net at U3. (X): now also U1.2
- new net: U1. (GND), U2. (X), U3. (X), U4.1 (VO)
- new net: BT1.2 (-), BZ1.2 (-), U1. (GND), U2. (X), U3. (X), U4.2 (GND)
- new net: U1.8 (SDA), U2. (X), U3. (X)
- new net: U1.9 (SCL), U2. (X), U3. (X)
- new net: BT1.1 (+), U4.3 (VI)
- now unconnected: U1. (GND), U1. (GND)
Other:
- moved on the sheet: BT1
Changed lines of the file:
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@@
+	)
+	(junction
+		(at 123.19 63.5)
+		(diameter 0)
+		(color 0 0 0 0)
 	)
 	(junction
@@
 	)
 	(junction
-		(at 127 67.31)
+		(at 138.43 55.88)
 		(diameter 0)
 		(color 0 0 0 0)
 	)
 	(junction
-		(at 123.19 71.12)
+		(at 127 67.31)
 		(diameter 0)
 		(color 0 0 0 0)
@@
 	(wire
 		(pts
+			(xy 123.19 63.5) (xy 130.81 63.5)
+		)
+		(stroke
+			(width 0)
+			(type default)
+		)
+	)
+	(wire
+		(pts
+			(xy 146.05 63.5) (xy 149.86 63.5)
+		)
+		(stroke
+			(width 0)
+			(type default)
+		)
+	)
+	(wire
+		(pts
 			(xy 127 67.31) (xy 127 116.84)
 		)
@@
 	(wire
 		(pts
-			(xy 123.19 71.12) (xy 135.89 71.12)
-		)
-		(stroke
-			(width 0)
-			(type default)
-		)
-	)
-	(wire
-		(pts
 			(xy 64.77 128.27) (xy 163.83 128.27)
 		)
@@
 	(wire
 		(pts
-			(xy 102.87 71.12) (xy 123.19 71.12)
-		)
-		(stroke
-			(width 0)
-			(type default)
-		)
-	)
-	(wire
-		(pts
 			(xy 76.2 82.55) (xy 72.39 82.55)
 		)
@@
 	(wire
 		(pts
+			(xy 138.43 55.88) (xy 127 55.88)
+		)
+		(stroke
+			(width 0)
+			(type default)
+		)
+	)
+	(wire
+		(pts
 			(xy 194.31 128.27) (xy 194.31 111.76)
 		)
@@
 	(wire
 		(pts
+			(xy 127 55.88) (xy 127 67.31)
+		)
+		(stroke
+			(width 0)
+			(type default)
+		)
+	)
+	(wire
+		(pts
 			(xy 186.69 116.84) (xy 156.21 116.84)
 		)
@@
 	(wire
 		(pts
+			(xy 138.43 55.88) (xy 157.48 55.88)
+		)
+		(stroke
+			(width 0)
+			(type default)
+		)
+	)
+	(wire
+		(pts
 			(xy 68.58 78.74) (xy 68.58 124.46)
 		)
@@
 	(wire
 		(pts
+			(xy 157.48 55.88) (xy 157.48 63.5)
+		)
+		(stroke
+			(width 0)
+			(type default)
+		)
+	)
+	(wire
+		(pts
 			(xy 199.39 138.43) (xy 186.69 138.43)
 		)
@@
 	(wire
 		(pts
-			(xy 135.89 71.12) (xy 135.89 67.31)
-		)
-		(stroke
-			(width 0)
-			(type default)
-		)
-	)
-	(wire
-		(pts
-			(xy 135.89 67.31) (xy 134.62 67.31)
-		)
-		(stroke
-			(width 0)
-			(type default)
-		)
-	)
-	(wire
-		(pts
-			(xy 123.19 71.12) (xy 123.19 120.65)
+			(xy 123.19 63.5) (xy 123.19 120.65)
 		)
 		(stroke
@@
 		(pts
 			(xy 76.2 78.74) (xy 68.58 78.74)
+		)
+		(stroke
+			(width 0)
+			(type default)
+		)
+	)
+	(wire
+		(pts
+			(xy 102.87 63.5) (xy 123.19 63.5)
 		)
 		(stroke
@@
 	)
 	(symbol
+		(lib_id "Regulator_Linear:LM78L05_TO92")
+		(at 138.43 63.5 180)
+		(unit 1)
+		(exclude_from_sim no)
+		(in_bom yes)
+		(on_board yes)
+		(dnp no)
+		(property "Reference" "U4"
+			(at 138.43 66.802 0)
+			(effects
+				(font
+					(size 1.27 1.27)
+				)
+			)
+		)
+		(property "Value" "LM78L05_TO92"
+			(at 138.43 69.342 0)
+			(effects
+				(font
+					(size 1.27 1.27)
+				)
+			)
+		)
+		(property "Footprint" "Package_TO_SOT_THT:TO-92_Inline"
+			(at 138.43 69.215 0)
+			(effects
+				(font
+					(size 1.27 1.27)
+					(italic yes)
+				)
+				(hide yes)
+			)
+		)
+		(property "Datasheet" "https://www.onsemi.com/pub/Collateral/MC78L06A-D.pdf"
+			(at 138.43 62.23 0)
+			(effects
+				(font
+					(size 1.27 1.27)
+				)
+				(hide yes)
+			)
+		)
+		(property "Description" "Positive 100mA 30V Linear Regulator, Fixed Output 5V, TO-92"
+			(at 138.43 63.5 0)
+			(effects
+				(font
+					(size 1.27 1.27)
+				)
+				(hide yes)
+			)
+		)
+		(pin "1"
+		)
+		(pin "3"
+		)
+		(pin "2"
+		)
+		(instances
+			(project ""
+				(path "/e697d9f0-6df0-4ad6-b7b8-3236f8a796fa"
+					(reference "U4")
+					(unit 1)
+				)
+			)
+		)
+	)
+	(symbol
 		(lib_id "Device:Battery_Cell")
-		(at 129.54 67.31 270)
+		(at 154.94 63.5 90)
 		(unit 1)
 		(exclude_from_sim no)
@@
 		(dnp no)
 		(property "Reference" "BT1"
-			(at 131.3815 59.69 90)
-			(effects
-				(font
-					(size 1.27 1.27)
-				)
-			)
-		)
-		(property "Value" "3V"
-			(at 131.3815 62.23 90)
+			(at 153.162 67.31 90)
+			(effects
+				(font
+					(size 1.27 1.27)
+				)
+			)
+		)
+		(property "Value" "12V"
+			(at 153.162 69.596 90)
 			(effects
 				(font
@@
 		)
 		(property "Footprint" ""
-			(at 131.064 67.31 90)
+			(at 153.416 63.5 90)
 			(effects
 				(font
@@
 		)
 		(property "Datasheet" "~"
-			(at 131.064 67.31 90)
+			(at 153.416 63.5 90)
 			(effects
 				(font
@@
 		)
 		(property "Description" "Single-cell battery"
-			(at 129.54 67.31 0)
-			(effects
-				(font
+			(at 154.94 63.5 0)
+			(effects
+				(font
